Commit message: added extra sensors to urdf

File: share/urdf/pepper.urdf (robot description, URDF)
Before this commit: robot JulietteY20MP, 84 links, 83 joints
Links:
- added link imu0
- added link sick_laser_front
- added link sick_laser_rear
Joints:
- added joint SickLaser/front: type fixed, parent Tibia, child sick_laser_front, origin xyz=0.245 0.0 -0.1 rpy=0 0 0, axis 0 0 0
- added joint SickLaser/rear: type fixed, parent Tibia, child sick_laser_rear, origin xyz=-0.245 0.0 -0.1 rpy=0 0 3.14159, axis 0 0 0
- added joint visensor_center: type fixed, parent Head, child imu0, origin xyz=-0.25 0.039 0 rpy=0 0 0, axis 0 0 0

Commit message: add realsense tf to pepper urdf

File: share/urdf/pepper.urdf (robot description, URDF)
Before this commit: robot JulietteY20MP, 87 links, 86 joints
Links:
- added link camera_link
Joints:
- added joint realsense: type fixed, parent Head, child camera_link, origin xyz=0.0715 0.0175 0.195 rpy=0 0 0, axis 0 0 0

Commit message: update lidar and realsense tf, currently best values

File: share/urdf/pepper.urdf (robot description, URDF)
Before this commit: robot JulietteY20MP, 88 links, 87 joints
Joints:
- joint SickLaser/front: origin xyz=0.245 0.0 -0.1 rpy=0 0 0 -> xyz=0.252 0.0 -0.1 rpy=0 0 -0.005
- joint SickLaser/rear: origin xyz=-0.245 0.0 -0.1 rpy=0 0 3.14159 -> xyz=-0.244 0.0 -0.1 rpy=0 0 3.14459
- joint realsense: origin xyz=0.0715 0.0175 0.195 rpy=0 0 0 -> xyz=0.0715 0.0175 0.195 rpy=0 0.07 0
